Commit message: Imported upstream version '0.1.1' of 'upstream'

File: dingo_description/urdf/accessories.urdf.xacro (robot description, xacro)
@@ -9,18 +9,13 @@
     dingo_base/launch/base.launch
   -->
-  <!-- If enabled, generate the LASER payload (by default, a SICK LMS111). -->
+  <!--
+    Add a lidar sensor.  By default this is a SICK LMS1xx but can be changed with the
+    DINGO_LASER_MODEL environment variable. Valid model designations are:
+    - lms1xx (default) :: SICK LMS1xx
+    - ust10            :: Hokuyo UST10
+  -->
   <xacro:if value="$(optenv DINGO_LASER 0)">
-    <xacro:if value="$(optenv DINGO_LASER_HOKUYO 0)">
-      <xacro:include filename="$(find dingo_description)/urdf/accessories/hokuyo_ust10.urdf.xacro" />
-      <xacro:hokuyo_ust10_mount prefix="$(optenv DINGO_LASER_MOUNT front)"
-                          topic="$(optenv DINGO_LASER_TOPIC front/scan)" />
-      <joint name="$(optenv DINGO_LASER_MOUNT front)_laser_mount_joint" type="fixed">
-        <origin xyz="$(optenv DINGO_LASER_OFFSET 0.11 0 0)"
-                rpy="$(optenv DINGO_LASER_RPY 0 0 0)" />
-        <parent link="$(optenv DINGO_LASER_MOUNT front)_mount" />
-        <child link="$(optenv DINGO_LASER_MOUNT front)_laser_mount" />
-      </joint>
-    </xacro:if>
-    <xacro:unless value="$(optenv DINGO_LASER_HOKUYO 0)">
+    <xacro:property name="lidar_model" value="$(optenv DINGO_LASER_MODEL lms1xx)" />
+    <xacro:if value="${lidar_model == 'lms1xx'}">
       <xacro:include filename="$(find dingo_description)/urdf/accessories/sick_lms1xx_mount.urdf.xacro" />
       <xacro:sick_lms1xx_mount prefix="$(optenv DINGO_LASER_MOUNT front)"
@@ -32,5 +27,31 @@
         <child link="$(optenv DINGO_LASER_MOUNT front)_laser_mount" />
       </joint>
-    </xacro:unless>
+    </xacro:if>
+    <xacro:if value="${lidar_model == 'ust10'}">
+      <xacro:include filename="$(find dingo_description)/urdf/accessories/hokuyo_ust10.urdf.xacro" />
+      <xacro:hokuyo_ust10_mount prefix="$(optenv DINGO_LASER_MOUNT front)"
+                          topic="$(optenv DINGO_LASER_TOPIC front/scan)" />
+      <joint name="$(optenv DINGO_LASER_MOUNT front)_laser_mount_joint" type="fixed">
+        <origin xyz="$(optenv DINGO_LASER_OFFSET 0 0 0)"
+                rpy="$(optenv DINGO_LASER_RPY 0 0 0)" />
+        <parent link="$(optenv DINGO_LASER_MOUNT front)_mount" />
+        <child link="$(optenv DINGO_LASER_MOUNT front)_laser_mount" />
+      </joint>
+    </xacro:if>
+  </xacro:if>
+  <!--
+    Add an Intel RealSense family camera.  By default this is a D435, but can be changed with the
+    DINGO_REALSENSE_MODEL environment variable. Valid model designations are:
+    - d435 (default)
+    - d435i
+    - d415
+    - d455
+    - l515
+  -->
+  <xacro:if value="$(optenv DINGO_REALSENSE 0)">
+    <include filename="$(find dingo_description)/urdf/accessories/intel_realsense.urdf.xacro" />
+    <xacro:realsense_sensor rs_model="$(optenv DINGO_REALSENSE_MODEL d435)"
+                            prefix="$(optenv DINGO_REALSENSE_MOUNT front)"
+                            topic="$(optenv DINGO_REALSENSE_TOPIC realsense)" />
   </xacro:if>
 </robot>

Commit message: Imported upstream version '0.1.11' of 'upstream'

File: dingo_description/urdf/accessories.urdf.xacro (robot description, xacro)
@@ -11,4 +11,5 @@
   <xacro:include filename="$(find dingo_description)/urdf/accessories/sick_lms1xx_mount.urdf.xacro" />
   <xacro:include filename="$(find dingo_description)/urdf/accessories/hokuyo_ust10.urdf.xacro" />
+  <xacro:include filename="$(find dingo_description)/urdf/accessories/hdl32_mount.urdf.xacro" />
   <xacro:include filename="$(find dingo_description)/urdf/accessories/vlp16_mount.urdf.xacro" />
   <!--
@@ -19,23 +20,47 @@
   -->
   <xacro:if value="$(optenv DINGO_LASER 0)">
+    <xacro:property name="mount" value="$(optenv DINGO_LASER_MOUNT front)" />
+    <xacro:property name="topic" value="$(optenv DINGO_LASER_TOPIC front/scan)" />
+    <xacro:property name="tower" value="$(optenv DINGO_LASER_TOWER 1)" />
+    <xacro:property name="prefix" value="$(optenv DINGO_LASER_PREFIX ${mount})" />
+    <xacro:property name="parent" value="$(optenv DINGO_LASER_PARENT ${mount}_mount)" />
     <xacro:property name="lidar_model" value="$(optenv DINGO_LASER_MODEL lms1xx)" />
+    <!-- SICK LMS1xx -->
     <xacro:if value="${lidar_model == 'lms1xx'}">
-      <xacro:sick_lms1xx_mount prefix="$(optenv DINGO_LASER_MOUNT front)"
-                         topic="$(optenv DINGO_LASER_TOPIC front/scan)"/>
-      <joint name="$(optenv DINGO_LASER_MOUNT front)_laser_mount_joint" type="fixed">
+      <!-- Mount Enabled -->
+      <xacro:if value="${tower}">
+        <xacro:sick_lms1xx_mount prefix="${prefix}" topic="${topic}"/>
+        <joint name="${prefix}_laser_mount_joint" type="fixed">
+          <origin xyz="$(optenv DINGO_LASER_OFFSET 0 0 0)"
+                  rpy="$(optenv DINGO_LASER_RPY 0 0 0)" />
+          <parent link="${parent}" />
+          <child link="${prefix}_laser_mount" />
+        </joint>
+      </xacro:if>
+      <!-- Mount Disabled -->
+      <xacro:unless value="${tower}">
+        <xacro:sick_lms1xx frame="${prefix}_laser" topic="${topic}" />
+        <link name="${prefix}_laser_base"/>
+        <joint name="${prefix}_laser_base_joint" type="fixed">
+          <origin xyz="$(optenv DINGO_LASER_OFFSET 0 0 0)"
+                  rpy="$(optenv DINGO_LASER_RPY 0 0 0)"/>
+          <parent link="${parent}"/>
+          <child link="${prefix}_laser_base"/>
+        </joint>
+        <joint name="${prefix}_laser_joint" type="fixed">
+          <origin xyz="0 0 0.116" rpy="0 0 0"/>
+          <parent link="${prefix}_laser_base"/>
+          <child link="${prefix}_laser"/>
+        </joint>
+      </xacro:unless>
+    </xacro:if>
+    <!-- Hokuyo UST10 -->
+    <xacro:if value="${lidar_model == 'ust10'}">
+      <xacro:hokuyo_ust10_mount prefix="${prefix}" topic="${topic}" />
+      <joint name="${prefix}_laser_mount_joint" type="fixed">
         <origin xyz="$(optenv DINGO_LASER_OFFSET 0 0 0)"
                 rpy="$(optenv DINGO_LASER_RPY 0 0 0)" />
-        <parent link="$(optenv DINGO_LASER_MOUNT front)_mount" />
-        <child link="$(optenv DINGO_LASER_MOUNT front)_laser_mount" />
-      </joint>
-    </xacro:if>
-    <xacro:if value="${lidar_model == 'ust10'}">
-      <xacro:hokuyo_ust10_mount prefix="$(optenv DINGO_LASER_MOUNT front)"
-                          topic="$(optenv DINGO_LASER_TOPIC front/scan)" />
-      <joint name="$(optenv DINGO_LASER_MOUNT front)_laser_mount_joint" type="fixed">
-        <origin xyz="$(optenv DINGO_LASER_OFFSET 0 0 0)"
-                rpy="$(optenv DINGO_LASER_RPY 0 0 0)" />
-        <parent link="$(optenv DINGO_LASER_MOUNT front)_mount" />
-        <child link="$(optenv DINGO_LASER_MOUNT front)_laser_mount" />
+        <parent link="${parent}" />
+        <child link="${prefix}_laser_mount" />
       </joint>
     </xacro:if>
@@ -43,23 +68,47 @@
   <!-- Add the secondary lidar, same format as the first, but on the rear -->
   <xacro:if value="$(optenv DINGO_LASER_SECONDARY 0)">
-    <xacro:property name="lidar2_model" value="$(optenv DINGO_LASER_SECONDARY_MODEL lms1xx)" />
-    <xacro:if value="${lidar2_model == 'lms1xx'}">
-      <xacro:sick_lms1xx_mount prefix="$(optenv DINGO_LASER_SECONDARY_MOUNT rear)"
-                         topic="$(optenv DINGO_LASER_SECONDARY_TOPIC rear/scan)"/>
-      <joint name="$(optenv DINGO_LASER_SECONDARY_MOUNT rear)_laser_mount_joint" type="fixed">
+    <xacro:property name="mount" value="$(optenv DINGO_LASER_SECONDARY_MOUNT rear)" />
+    <xacro:property name="topic" value="$(optenv DINGO_LASER_SECONDARY_TOPIC rear/scan)" />
+    <xacro:property name="tower" value="$(optenv DINGO_LASER_SECONDARY_TOWER 1)" />
+    <xacro:property name="prefix" value="$(optenv DINGO_LASER_SECONDARY_PREFIX ${mount})" />
+    <xacro:property name="parent" value="$(optenv DINGO_LASER_SECONDARY_PARENT ${mount}_mount)" />
+    <xacro:property name="lidar_model" value="$(optenv DINGO_LASER_SECONDARY_MODEL lms1xx)" />
+    <!-- Secondary SICK LMS1xx -->
+    <xacro:if value="${lidar_model == 'lms1xx'}">
+      <!-- Mount Enabled -->
+      <xacro:if value="${tower}">
+        <xacro:sick_lms1xx_mount prefix="${prefix}" topic="${topic}"/>
+        <joint name="${prefix}_laser_mount_joint" type="fixed">
+          <origin xyz="$(optenv DINGO_LASER_SECONDARY_OFFSET 0 0 0)"
+                  rpy="$(optenv DINGO_LASER_SECONDARY_RPY 0 0 ${M_PI})" />
+          <parent link="${parent}" />
+          <child link="${prefix}_laser_mount" />
+        </joint>
+      </xacro:if>
+      <!-- Mount Disabled -->
+      <xacro:unless value="${tower}">
+        <xacro:sick_lms1xx frame="${prefix}_laser" topic="${topic}" />
+        <link name="${prefix}_laser_base"/>
+        <joint name="${prefix}_laser_base_joint" type="fixed">
+          <origin xyz="$(optenv DINGO_LASER_SECONDARY_OFFSET 0 0 0)"
+                  rpy="$(optenv DINGO_LASER_SECONDARY_RPY 0 0 ${M_PI})" />
+          <parent link="${parent}"/>
+          <child link="${prefix}_laser_base"/>
+        </joint>
+        <joint name="${prefix}_laser_joint" type="fixed">
+          <origin xyz="0 0 0.116" rpy="0 0 0"/>
+          <parent link="${prefix}_laser_base"/>
+          <child link="${prefix}_laser"/>
+        </joint>
+      </xacro:unless>
+    </xacro:if>
+    <!-- Secondary Hokuyo UST10 -->
+    <xacro:if value="${lidar_model == 'ust10'}">
+      <xacro:hokuyo_ust10_mount prefix="${prefix}" topic="${topic}" />
+      <joint name="${prefix}_laser_mount_joint" type="fixed">
         <origin xyz="$(optenv DINGO_LASER_SECONDARY_OFFSET 0 0 0)"
                 rpy="$(optenv DINGO_LASER_SECONDARY_RPY 0 0 ${M_PI})" />
-        <parent link="$(optenv DINGO_LASER_SECONDARY_MOUNT rear)_mount" />
-        <child link="$(optenv DINGO_LASER_SECONDARY_MOUNT rear)_laser_mount" />
-      </joint>
-    </xacro:if>
-    <xacro:if value="${lidar2_model == 'ust10'}">
-      <xacro:hokuyo_ust10_mount prefix="$(optenv DINGO_LASER_SECONDARY_MOUNT rear)"
-                          topic="$(optenv DINGO_LASER_SECONDARY_TOPIC rear/scan)" />
-      <joint name="$(optenv DINGO_LASER_SECONDARY_MOUNT rear)_laser_mount_joint" type="fixed">
-        <origin xyz="$(optenv DINGO_LASER_SECONDARY_OFFSET 0 0 0)"
-                rpy="$(optenv DINGO_LASER_SECONDARY_RPY 0 0 ${M_PI})" />
-        <parent link="$(optenv DINGO_LASER_SECONDARY_MOUNT rear)_mount" />
-        <child link="$(optenv DINGO_LASER_SECONDARY_MOUNT rear)_laser_mount" />
+        <parent link="${parent}" />
+        <child link="${prefix}_laser_mount" />
       </joint>
     </xacro:if>
@@ -71,12 +120,22 @@
   -->
   <xacro:if value="$(optenv DINGO_LASER_3D 0)">
+    <xacro:property name="mount" value="$(optenv DINGO_LASER_3D_MOUNT front)" />
+    <xacro:property name="topic" value="$(optenv DINGO_LASER_3D_TOPIC front/points)" />
+    <xacro:property name="tower" value="$(optenv DINGO_LASER_3D_TOWER 1)" />
+    <xacro:property name="angle" value="$(optenv DINGO_LASER_3D_ANGLE 0)" />
+    <xacro:property name="prefix" value="$(optenv DINGO_LASER_3D_PREFIX ${mount})" />
+    <xacro:property name="parent" value="$(optenv DINGO_LASER_3D_PARENT ${mount}_mount)" />
     <xacro:property name="lidar_3d_model" value="$(optenv DINGO_LASER_3D_MODEL vlp16)" />
+    <!-- Velodyne VLP16 -->
     <xacro:if value="${lidar_3d_model == 'vlp16'}">
-      <xacro:vlp16_mount
-          prefix="$(optenv DINGO_LASER_3D_MOUNT front)"
-          parent_link="$(optenv DINGO_LASER_3D_MOUNT front)_mount"
-          topic="$(optenv DINGO_LASER_3D_TOPIC front/points)">
+      <xacro:vlp16_mount topic="${topic}" tower="${tower}" angle="${angle}" prefix="${prefix}" parent_link="${parent}" >
         <origin xyz="$(optenv DINGO_LASER_3D_OFFSET 0 0 0)" rpy="$(optenv DINGO_LASER_3D_RPY 0 0 0)" />
       </xacro:vlp16_mount>
+    </xacro:if>
+    <!-- Velodyne HDL-32E -->
+    <xacro:if value="${lidar_3d_model == 'hdl32e'}">
+      <xacro:hdl32e_mount topic="${topic}" tower="${tower}" angle="${angle}" prefix="${prefix}" parent_link="${parent}" >
+        <origin xyz="$(optenv DINGO_LASER_3D_OFFSET 0 0 0)" rpy="$(optenv DINGO_LASER_3D_RPY 0 0 0)" />
+      </xacro:hdl32e_mount>
     </xacro:if>
   </xacro:if>
@@ -96,3 +155,19 @@
                             topic="$(optenv DINGO_REALSENSE_TOPIC realsense)" />
   </xacro:if>
+  <!--
+    Add Microstrain IMU. By default the DINGO comes equipped with an IMU linked to "imu_link". These extra
+    optional microstrain IMU's will be added to another frame, by default, "microstrain_link".
+  -->
+  <xacro:if value="$(optenv DINGO_IMU_MICROSTRAIN 0)">
+    <xacro:property name="frame"  value="$(optenv DINGO_IMU_MICROSTRAIN_LINK microstrain_link)"/>
+    <xacro:property name="parent" value="$(optenv DINGO_IMU_MICROSTRAIN_PARENT imu_link)"/>
+    <xacro:property name="xyz"    value="$(optenv DINGO_IMU_MICROSTRAIN_OFFSET 0 0 0)"/>
+    <xacro:property name="rpy"    value="$(optenv DINGO_IMU_MICROSTRAIN_RPY 0 0 0)"/>
+    <link name="${frame}" />
+    <joint name="${frame}_joint" type="fixed">
+      <parent link="${parent}" />
+      <child link="${frame}" />
+      <origin xyz="${xyz}" rpy="${rpy}" />
+    </joint>
+  </xacro:if>
 </robot>

File: dingo_description/urdf/accessories/vlp16_mount.urdf.xacro (robot description, xacro)
@@ -1,92 +1,99 @@
 <robot xmlns:xacro="http://wiki.ros.org/xacro">
   <xacro:include filename="$(find velodyne_description)/urdf/VLP-16.urdf.xacro" />
-  <xacro:macro name="vlp16_mount" params="prefix parent_link topic height:=0.1 *origin">
-    <link name="${prefix}_vlp16_mount" />
-    <link name="${prefix}_vlp16_plate">
-      <visual>
-        <geometry>
-          <box size="0.1 0.1 0.002" />
-        </geometry>
-        <material name="black" />
-        <origin xyz="0 0 -0.001" rpy="0 0 0" />
-      </visual>
-    </link>
-    <link name="${prefix}_vlp16_leg1">
-      <visual>
-        <geometry>
-          <cylinder length="${height}" radius="0.003" />
-        </geometry>
-        <material name="white">
-          <color rgba="1 1 1 1" />
-        </material>
-        <origin xyz="0 0 ${height/2}" rpy="0 0 0" />
-      </visual>
-    </link>
-    <link name="${prefix}_vlp16_leg2">
-      <visual>
-        <geometry>
-          <cylinder length="${height}" radius="0.003" />
-        </geometry>
-        <material name="white">
-          <color rgba="1 1 1 1" />
-        </material>
-        <origin xyz="0 0 ${height/2}" rpy="0 0 0" />
-      </visual>
-    </link>
-    <link name="${prefix}_vlp16_leg3">
-      <visual>
-        <geometry>
-          <cylinder length="${height}" radius="0.003" />
-        </geometry>
-        <material name="white">
-          <color rgba="1 1 1 1" />
-        </material>
-        <origin xyz="0 0 ${height/2}" rpy="0 0 0" />
-      </visual>
-    </link>
-    <link name="${prefix}_vlp16_leg4">
-      <visual>
-        <geometry>
-          <cylinder length="${height}" radius="0.003" />
-        </geometry>
-        <material name="white">
-          <color rgba="1 1 1 1" />
-        </material>
-        <origin xyz="0 0 ${height/2}" rpy="0 0 0" />
-      </visual>
-    </link>
-    <joint name="${prefix}_vlp16_mount_joint" type="fixed">
-      <parent link="${parent_link}" />
-      <child link="${prefix}_vlp16_mount" />
-      <xacro:insert_block name="origin" />
-    </joint>
-    <joint name="${prefix}_vlp16_leg1_joint" type="fixed">
-      <parent link="${prefix}_mount" />
-      <child link="${prefix}_vlp16_leg1" />
-      <origin xyz="0.05 0.05 0" rpy="0 0 0" />
-    </joint>
-    <joint name="${prefix}_vlp16_leg2_joint" type="fixed">
-      <parent link="${prefix}_mount" />
-      <child link="${prefix}_vlp16_leg2" />
-      <origin xyz="0.05 -0.05 0" rpy="0 0 0" />
-    </joint>
-    <joint name="${prefix}_vlp16_leg3_joint" type="fixed">
-      <parent link="${prefix}_mount" />
-      <child link="${prefix}_vlp16_leg3" />
-      <origin xyz="-0.05 0.05 0" rpy="0 0 0" />
-    </joint>
-    <joint name="${prefix}_vlp16_leg4_joint" type="fixed">
-      <parent link="${prefix}_mount" />
-      <child link="${prefix}_vlp16_leg4" />
-      <origin xyz="-0.05 -0.05 0" rpy="0 0 0" />
-    </joint>
-    <joint name="${prefix}_vlp16_plate_joint" type="fixed">
-      <parent link="${prefix}_vlp16_mount" />
-      <child link="${prefix}_vlp16_plate" />
-      <origin xyz="0 0 ${height}" rpy="0 0 0" />
-    </joint>
-    <xacro:VLP-16 parent="${prefix}_vlp16_plate" topic="${topic}">
-      <origin xyz="0 0 0" rpy="0 0 0" />
-    </xacro:VLP-16>
+  <xacro:macro name="vlp16_mount" params="prefix parent_link topic tower angle:=0 height:=0.1 *origin">
+    <xacro:if value="${tower}">
+      <link name="${prefix}_vlp16_mount" />
+      <link name="${prefix}_vlp16_plate">
+        <visual>
+          <geometry>
+            <box size="0.1 0.1 0.002" />
+          </geometry>
+          <material name="black" />
+          <origin xyz="0 0 -0.001" rpy="0 0 0" />
+        </visual>
+      </link>
+      <link name="${prefix}_vlp16_leg1">
+        <visual>
+          <geometry>
+            <cylinder length="${height}" radius="0.003" />
+          </geometry>
+          <material name="white">
+            <color rgba="1 1 1 1" />
+          </material>
+          <origin xyz="0 0 ${height/2}" rpy="0 0 0" />
+        </visual>
+      </link>
+      <link name="${prefix}_vlp16_leg2">
+        <visual>
+          <geometry>
+            <cylinder length="${height}" radius="0.003" />
+          </geometry>
+          <material name="white">
+            <color rgba="1 1 1 1" />
+          </material>
+          <origin xyz="0 0 ${height/2}" rpy="0 0 0" />
+        </visual>
+      </link>
+      <link name="${prefix}_vlp16_leg3">
+        <visual>
+          <geometry>
+            <cylinder length="${height}" radius="0.003" />
+          </geometry>
+          <material name="white">
+            <color rgba="1 1 1 1" />
+          </material>
+          <origin xyz="0 0 ${height/2}" rpy="0 0 0" />
+        </visual>
+      </link>
+      <link name="${prefix}_vlp16_leg4">
+        <visual>
+          <geometry>
+            <cylinder length="${height}" radius="0.003" />
+          </geometry>
+          <material name="white">
+            <color rgba="1 1 1 1" />
+          </material>
+          <origin xyz="0 0 ${height/2}" rpy="0 0 0" />
+        </visual>
+      </link>
+      <joint name="${prefix}_vlp16_mount_joint" type="fixed">
+        <parent link="${parent_link}" />
+        <child link="${prefix}_vlp16_mount" />
+        <xacro:insert_block name="origin" />
+      </joint>
+      <joint name="${prefix}_vlp16_leg1_joint" type="fixed">
+        <parent link="${prefix}_vlp16_mount" />
+        <child link="${prefix}_vlp16_leg1" />
+        <origin xyz="0.05 0.05 0" rpy="0 0 0" />
+      </joint>
+      <joint name="${prefix}_vlp16_leg2_joint" type="fixed">
+        <parent link="${prefix}_vlp16_mount" />
+        <child link="${prefix}_vlp16_leg2" />
+        <origin xyz="0.05 -0.05 0" rpy="0 0 0" />
+      </joint>
+      <joint name="${prefix}_vlp16_leg3_joint" type="fixed">
+        <parent link="${prefix}_vlp16_mount" />
+        <child link="${prefix}_vlp16_leg3" />
+        <origin xyz="-0.05 0.05 0" rpy="0 0 0" />
+      </joint>
+      <joint name="${prefix}_vlp16_leg4_joint" type="fixed">
+        <parent link="${prefix}_vlp16_mount" />
+        <child link="${prefix}_vlp16_leg4" />
+        <origin xyz="-0.05 -0.05 0" rpy="0 0 0" />
+      </joint>
+      <joint name="${prefix}_vlp16_plate_joint" type="fixed">
+        <parent link="${prefix}_vlp16_mount" />
+        <child link="${prefix}_vlp16_plate" />
+        <origin xyz="0 0 ${height}" rpy="0 0 0" />
+      </joint>
+      <xacro:VLP-16 parent="${prefix}_vlp16_plate" topic="${topic}">
+        <origin xyz="0 0 0" rpy="0 0 ${angle}" />
+      </xacro:VLP-16>
+    </xacro:if>
+    <xacro:unless value="${tower}">
+      <xacro:VLP-16 parent="${parent_link}" topic="${topic}">
+        <xacro:insert_block name="origin" />
+      </xacro:VLP-16>
+    </xacro:unless>
   </xacro:macro>
 </robot>
