Commit message: Imported upstream version '0.2.0' of 'upstream'

File: dingo_description/urdf/accessories.urdf.xacro (robot description, xacro)
@@ -227,4 +227,36 @@
     </xacro:realsense_sensor>
   </xacro:if>
+  <!-- BlackflyS Camera Primary and Secondary -->
+  <xacro:include filename="$(find dingo_description)/urdf/accessories/flir_blackfly_mount.urdf.xacro"/>
+  <xacro:arg name="blackfly_enabled"                  default="$(optenv DINGO_BLACKFLY 0)"/>
+  <xacro:arg name="blackfly_mount_enabled"            default="$(optenv DINGO_BLACKFLY_MOUNT_ENABLED 1)"/>
+  <xacro:arg name="blackfly_mount_angle"              default="$(optenv DINGO_BLACKFLY_MOUNT_ANGLE 0)"/>
+  <xacro:arg name="blackfly_prefix"                   default="$(optenv DINGO_BLACKFLY_PREFIX blackfly)"/>
+  <xacro:arg name="blackfly_parent"                   default="$(optenv DINGO_BLACKFLY_PARENT top_plate_link)"/>
+  <xacro:arg name="blackfly_xyz"                      default="$(optenv DINGO_BLACKFLY_XYZ 0 0 0)"/>
+  <xacro:arg name="blackfly_rpy"                      default="$(optenv DINGO_BLACKFLY_RPY 0 0 0)"/>
+  <xacro:arg name="blackfly_secondary_enabled"        default="$(optenv DINGO_BLACKFLY_SECONDARY 0)"/>
+  <xacro:arg name="blackfly_secondary_mount_enabled"  default="$(optenv DINGO_BLACKFLY_SECONDARY_MOUNT_ENABLED 1)"/>
+  <xacro:arg name="blackfly_secondary_mount_angle"    default="$(optenv DINGO_BLACKFLY_SECONDARY_MOUNT_ANGLE 0)"/>
+  <xacro:arg name="blackfly_secondary_prefix"         default="$(optenv DINGO_BLACKFLY_SECONDARY_PREFIX blackfly_secondary)"/>
+  <xacro:arg name="blackfly_secondary_parent"         default="$(optenv DINGO_BLACKFLY_SECONDARY_PARENT top_plate_link)"/>
+  <xacro:arg name="blackfly_secondary_xyz"            default="$(optenv DINGO_BLACKFLY_SECONDARY_XYZ 0 0 0)"/>
+  <xacro:arg name="blackfly_secondary_rpy"            default="$(optenv DINGO_BLACKFLY_SECONDARY_RPY 0 0 0)"/>
+  <xacro:if value="$(arg blackfly_enabled)">
+    <xacro:flir_blackfly_mount prefix="$(arg blackfly_prefix)"
+                                parent="$(arg blackfly_parent)"
+                                mount_enabled="$(arg blackfly_mount_enabled)"
+                                mount_angle="$(arg blackfly_mount_angle)">
+      <origin xyz="$(arg blackfly_xyz)" rpy="$(arg blackfly_rpy)"/>
+    </xacro:flir_blackfly_mount>
+  </xacro:if>
+  <xacro:if value="$(arg blackfly_secondary_enabled)">
+    <xacro:flir_blackfly_mount prefix="$(arg blackfly_secondary_prefix)"
+                                parent="$(arg blackfly_secondary_parent)"
+                                mount_enabled="$(arg blackfly_secondary_mount_enabled)"
+                                mount_angle="$(arg blackfly_secondary_mount_angle)">
+      <origin xyz="$(arg blackfly_secondary_xyz)" rpy="$(arg blackfly_secondary_rpy)"/>
+    </xacro:flir_blackfly_mount>
+  </xacro:if>
   <!--
     Add Microstrain IMU. By default the DINGO comes equipped with an IMU linked to "imu_link". These extra

File: dingo_description/urdf/pacs.urdf.xacro (robot description, xacro)
@@ -136,5 +136,6 @@
     Riser: adds riser with posts
   -->
-  <xacro:macro name="riser" params="height parent *origin">
+  <xacro:macro name="riser" params="level parent *origin">
+    <xacro:property name="height" value="${level * 0.1}"/>
     <!-- Quad Posts -->
     <xacro:quad_post parent="chassis_link" prefix="riser_base_link" length="0.16" width="0.08" height="${height-0.00635}">
@@ -163,5 +164,5 @@
     </joint>
     <!-- Mounts -->
-    <xacro:mounts parent="riser" level="1"/>
+    <xacro:mounts parent="riser" level="${riser}"/>
   </xacro:macro>
   <!--
@@ -286,5 +287,5 @@
       </xacro:if>
       <xacro:if value="${riser}">
-        <xacro:riser height="0.100" parent="base_link">
+        <xacro:riser level="${riser}" parent="base_link">
           <origin xyz="${riser_x} 0 0.069"/>
         </xacro:riser>

Commit message: Imported upstream version '0.1.12' of 'upstream'

File: dingo_description/urdf/accessories.urdf.xacro (robot description, xacro)
@@ -227,36 +227,4 @@
     </xacro:realsense_sensor>
   </xacro:if>
-  <!-- BlackflyS Camera Primary and Secondary -->
-  <xacro:include filename="$(find dingo_description)/urdf/accessories/flir_blackfly_mount.urdf.xacro"/>
-  <xacro:arg name="blackfly_enabled"                  default="$(optenv DINGO_BLACKFLY 0)"/>
-  <xacro:arg name="blackfly_mount_enabled"            default="$(optenv DINGO_BLACKFLY_MOUNT_ENABLED 1)"/>
-  <xacro:arg name="blackfly_mount_angle"              default="$(optenv DINGO_BLACKFLY_MOUNT_ANGLE 0)"/>
-  <xacro:arg name="blackfly_prefix"                   default="$(optenv DINGO_BLACKFLY_PREFIX blackfly)"/>
-  <xacro:arg name="blackfly_parent"                   default="$(optenv DINGO_BLACKFLY_PARENT top_plate_link)"/>
-  <xacro:arg name="blackfly_xyz"                      default="$(optenv DINGO_BLACKFLY_XYZ 0 0 0)"/>
-  <xacro:arg name="blackfly_rpy"                      default="$(optenv DINGO_BLACKFLY_RPY 0 0 0)"/>
-  <xacro:arg name="blackfly_secondary_enabled"        default="$(optenv DINGO_BLACKFLY_SECONDARY 0)"/>
-  <xacro:arg name="blackfly_secondary_mount_enabled"  default="$(optenv DINGO_BLACKFLY_SECONDARY_MOUNT_ENABLED 1)"/>
-  <xacro:arg name="blackfly_secondary_mount_angle"    default="$(optenv DINGO_BLACKFLY_SECONDARY_MOUNT_ANGLE 0)"/>
-  <xacro:arg name="blackfly_secondary_prefix"         default="$(optenv DINGO_BLACKFLY_SECONDARY_PREFIX blackfly_secondary)"/>
-  <xacro:arg name="blackfly_secondary_parent"         default="$(optenv DINGO_BLACKFLY_SECONDARY_PARENT top_plate_link)"/>
-  <xacro:arg name="blackfly_secondary_xyz"            default="$(optenv DINGO_BLACKFLY_SECONDARY_XYZ 0 0 0)"/>
-  <xacro:arg name="blackfly_secondary_rpy"            default="$(optenv DINGO_BLACKFLY_SECONDARY_RPY 0 0 0)"/>
-  <xacro:if value="$(arg blackfly_enabled)">
-    <xacro:flir_blackfly_mount prefix="$(arg blackfly_prefix)"
-                                parent="$(arg blackfly_parent)"
-                                mount_enabled="$(arg blackfly_mount_enabled)"
-                                mount_angle="$(arg blackfly_mount_angle)">
-      <origin xyz="$(arg blackfly_xyz)" rpy="$(arg blackfly_rpy)"/>
-    </xacro:flir_blackfly_mount>
-  </xacro:if>
-  <xacro:if value="$(arg blackfly_secondary_enabled)">
-    <xacro:flir_blackfly_mount prefix="$(arg blackfly_secondary_prefix)"
-                                parent="$(arg blackfly_secondary_parent)"
-                                mount_enabled="$(arg blackfly_secondary_mount_enabled)"
-                                mount_angle="$(arg blackfly_secondary_mount_angle)">
-      <origin xyz="$(arg blackfly_secondary_xyz)" rpy="$(arg blackfly_secondary_rpy)"/>
-    </xacro:flir_blackfly_mount>
-  </xacro:if>
   <!--
     Add Microstrain IMU. By default the DINGO comes equipped with an IMU linked to "imu_link". These extra

File: dingo_description/urdf/pacs.urdf.xacro (robot description, xacro)
@@ -136,6 +136,5 @@
     Riser: adds riser with posts
   -->
-  <xacro:macro name="riser" params="level parent *origin">
-    <xacro:property name="height" value="${level * 0.1}"/>
+  <xacro:macro name="riser" params="height parent *origin">
     <!-- Quad Posts -->
     <xacro:quad_post parent="chassis_link" prefix="riser_base_link" length="0.16" width="0.08" height="${height-0.00635}">
@@ -164,5 +163,5 @@
     </joint>
     <!-- Mounts -->
-    <xacro:mounts parent="riser" level="${riser}"/>
+    <xacro:mounts parent="riser" level="1"/>
   </xacro:macro>
   <!--
@@ -287,5 +286,5 @@
       </xacro:if>
       <xacro:if value="${riser}">
-        <xacro:riser level="${riser}" parent="base_link">
+        <xacro:riser height="0.100" parent="base_link">
           <origin xyz="${riser_x} 0 0.069"/>
         </xacro:riser>

Commit message: Imported upstream version '0.3.0' of 'upstream'

File: dingo_description/urdf/accessories.urdf.xacro (robot description, xacro)
@@ -227,4 +227,36 @@
     </xacro:realsense_sensor>
   </xacro:if>
+  <!-- BlackflyS Camera Primary and Secondary -->
+  <xacro:include filename="$(find dingo_description)/urdf/accessories/flir_blackfly_mount.urdf.xacro"/>
+  <xacro:arg name="blackfly_enabled"                  default="$(optenv DINGO_BLACKFLY 0)"/>
+  <xacro:arg name="blackfly_mount_enabled"            default="$(optenv DINGO_BLACKFLY_MOUNT_ENABLED 1)"/>
+  <xacro:arg name="blackfly_mount_angle"              default="$(optenv DINGO_BLACKFLY_MOUNT_ANGLE 0)"/>
+  <xacro:arg name="blackfly_prefix"                   default="$(optenv DINGO_BLACKFLY_PREFIX blackfly)"/>
+  <xacro:arg name="blackfly_parent"                   default="$(optenv DINGO_BLACKFLY_PARENT top_plate_link)"/>
+  <xacro:arg name="blackfly_xyz"                      default="$(optenv DINGO_BLACKFLY_XYZ 0 0 0)"/>
+  <xacro:arg name="blackfly_rpy"                      default="$(optenv DINGO_BLACKFLY_RPY 0 0 0)"/>
+  <xacro:arg name="blackfly_secondary_enabled"        default="$(optenv DINGO_BLACKFLY_SECONDARY 0)"/>
+  <xacro:arg name="blackfly_secondary_mount_enabled"  default="$(optenv DINGO_BLACKFLY_SECONDARY_MOUNT_ENABLED 1)"/>
+  <xacro:arg name="blackfly_secondary_mount_angle"    default="$(optenv DINGO_BLACKFLY_SECONDARY_MOUNT_ANGLE 0)"/>
+  <xacro:arg name="blackfly_secondary_prefix"         default="$(optenv DINGO_BLACKFLY_SECONDARY_PREFIX blackfly_secondary)"/>
+  <xacro:arg name="blackfly_secondary_parent"         default="$(optenv DINGO_BLACKFLY_SECONDARY_PARENT top_plate_link)"/>
+  <xacro:arg name="blackfly_secondary_xyz"            default="$(optenv DINGO_BLACKFLY_SECONDARY_XYZ 0 0 0)"/>
+  <xacro:arg name="blackfly_secondary_rpy"            default="$(optenv DINGO_BLACKFLY_SECONDARY_RPY 0 0 0)"/>
+  <xacro:if value="$(arg blackfly_enabled)">
+    <xacro:flir_blackfly_mount prefix="$(arg blackfly_prefix)"
+                                parent="$(arg blackfly_parent)"
+                                mount_enabled="$(arg blackfly_mount_enabled)"
+                                mount_angle="$(arg blackfly_mount_angle)">
+      <origin xyz="$(arg blackfly_xyz)" rpy="$(arg blackfly_rpy)"/>
+    </xacro:flir_blackfly_mount>
+  </xacro:if>
+  <xacro:if value="$(arg blackfly_secondary_enabled)">
+    <xacro:flir_blackfly_mount prefix="$(arg blackfly_secondary_prefix)"
+                                parent="$(arg blackfly_secondary_parent)"
+                                mount_enabled="$(arg blackfly_secondary_mount_enabled)"
+                                mount_angle="$(arg blackfly_secondary_mount_angle)">
+      <origin xyz="$(arg blackfly_secondary_xyz)" rpy="$(arg blackfly_secondary_rpy)"/>
+    </xacro:flir_blackfly_mount>
+  </xacro:if>
   <!--
     Add Microstrain IMU. By default the DINGO comes equipped with an IMU linked to "imu_link". These extra
@@ -233,5 +265,5 @@
   <xacro:if value="$(optenv DINGO_IMU_MICROSTRAIN 0)">
     <xacro:property name="frame"  value="$(optenv DINGO_IMU_MICROSTRAIN_LINK microstrain_link)"/>
-    <xacro:property name="parent" value="$(optenv DINGO_IMU_MICROSTRAIN_PARENT imu_link)"/>
+    <xacro:property name="parent" value="$(optenv DINGO_IMU_MICROSTRAIN_PARENT base_link)"/>
     <xacro:property name="xyz"    value="$(optenv DINGO_IMU_MICROSTRAIN_OFFSET 0 0 0)"/>
     <xacro:property name="rpy"    value="$(optenv DINGO_IMU_MICROSTRAIN_RPY 0 0 0)"/>

Commit message: Rebase from 'upstream'

File: dingo_description/urdf/accessories.urdf.xacro (robot description, xacro)
@@ -265,5 +265,5 @@
   <xacro:if value="$(optenv DINGO_IMU_MICROSTRAIN 0)">
     <xacro:property name="frame"  value="$(optenv DINGO_IMU_MICROSTRAIN_LINK microstrain_link)"/>
-    <xacro:property name="parent" value="$(optenv DINGO_IMU_MICROSTRAIN_PARENT imu_link)"/>
+    <xacro:property name="parent" value="$(optenv DINGO_IMU_MICROSTRAIN_PARENT base_link)"/>
     <xacro:property name="xyz"    value="$(optenv DINGO_IMU_MICROSTRAIN_OFFSET 0 0 0)"/>
     <xacro:property name="rpy"    value="$(optenv DINGO_IMU_MICROSTRAIN_RPY 0 0 0)"/>

Commit message: Imported upstream version '0.3.1' of 'upstream'

File: dingo_description/urdf/accessories.urdf.xacro (robot description, xacro)
@@ -9,4 +9,5 @@
     dingo_base/launch/base.launch
   -->
+  <xacro:include filename="$(find sick_tim)/urdf/sick_tim.urdf.xacro" />
   <xacro:include filename="$(find dingo_description)/urdf/accessories/sick_lms1xx_mount.urdf.xacro" />
   <xacro:include filename="$(find dingo_description)/urdf/accessories/hokuyo_ust10.urdf.xacro" />
@@ -17,4 +18,5 @@
     DINGO_LASER_MODEL environment variable. Valid model designations are:
     - lms1xx (default) :: SICK LMS1xx
+    - tim551           :: SICK TIM551
     - ust10            :: Hokuyo UST10
   -->
@@ -54,4 +56,14 @@
         </joint>
       </xacro:unless>
+    </xacro:if>
+    <!-- Sick TIM -->
+    <xacro:if value="${lidar_model == 'tim551'}">
+      <xacro:property name="prefix" value="$(optenv DINGO_LASER_PREFIX tim551)" />
+      <xacro:sick_tim551 name="${prefix}" ros_topic="${topic}"/>
+      <joint name="${prefix}_mount_link_joint" type="fixed">
+        <origin xyz="$(optenv DINGO_LASER_OFFSET 0 0 0)" rpy="$(optenv DINGO_LASER_RPY 0 0 0)"/>
+        <parent link="${parent}"/>
+        <child link="${prefix}_mount_link"/>
+      </joint>
     </xacro:if>
     <!-- Hokuyo UST10 -->
@@ -102,4 +114,14 @@
         </joint>
       </xacro:unless>
+    </xacro:if>
+    <!-- SICK Tim -->
+    <xacro:if value="${lidar_model == 'tim551'}">
+      <xacro:property name="prefix" value="$(optenv DINGO_LASER_SECONDARY_PREFIX tim551_2)" />
+      <xacro:sick_tim551 name="${prefix}" ros_topic="${topic}"/>
+      <joint name="${prefix}_mount_link_joint" type="fixed">
+        <origin xyz="$(optenv DINGO_LASER_SECONDARY_OFFSET 0 0 0)" rpy="$(optenv DINGO_LASER_SECONDARY_RPY 0 0 3.14159)"/>
+        <parent link="${parent}"/>
+        <child link="${prefix}_mount_link"/>
+      </joint>
     </xacro:if>
     <!-- Secondary Hokuyo UST10 -->

File: dingo_description/urdf/dingo-d.urdf.xacro (robot description, xacro)
@@ -169,42 +169,40 @@
       - rear
   -->
-  <xacro:unless value="${pacs_enabled}">
-    <link name="front_mount"/>
-    <link name="front_b_mount"/>
-    <link name="front_c_mount"/>
-    <link name="rear_mount"/>
-    <link name="rear_b_mount"/>
-    <link name="rear_c_mount"/>
-    <joint name="front_c_mount_joint" type="fixed">
-      <origin xyz="0.040 0 0.064263" rpy="0 0 0" />
-      <parent link="chassis_link"/>
-      <child link="front_c_mount" />
-    </joint>
-    <joint name="front_b_mount_joint" type="fixed">
-      <origin xyz="0.080 0 0" rpy="0 0 0" />
-      <parent link="front_c_mount"/>
-      <child link="front_b_mount" />
-    </joint>
-    <joint name="front_mount_joint" type="fixed">
-      <origin xyz="0.080 0 0" rpy="0 0 0" />
-      <parent link="front_b_mount"/>
-      <child link="front_mount" />
-    </joint>
-    <joint name="rear_c_mount_joint" type="fixed">
-      <origin xyz="-0.040 0 0.064263" rpy="0 0 0" />
-      <parent link="chassis_link"/>
-      <child link="rear_c_mount" />
-    </joint>
-    <joint name="rear_b_mount_joint" type="fixed">
-      <origin xyz="-0.080 0 0" rpy="0 0 0" />
-      <parent link="rear_c_mount"/>
-      <child link="rear_b_mount" />
-    </joint>
-    <joint name="rear_moint_joint" type="fixed">
-      <origin xyz="-0.080 0 0" rpy="0 0 0" />
-      <parent link="rear_b_mount"/>
-      <child link="rear_mount" />
-    </joint>
-  </xacro:unless>
+  <link name="front_mount"/>
+  <link name="front_b_mount"/>
+  <link name="front_c_mount"/>
+  <link name="rear_mount"/>
+  <link name="rear_b_mount"/>
+  <link name="rear_c_mount"/>
+  <joint name="front_c_mount_joint" type="fixed">
+    <origin xyz="0.040 0 0.064263" rpy="0 0 0" />
+    <parent link="chassis_link"/>
+    <child link="front_c_mount" />
+  </joint>
+  <joint name="front_b_mount_joint" type="fixed">
+    <origin xyz="0.080 0 0" rpy="0 0 0" />
+    <parent link="front_c_mount"/>
+    <child link="front_b_mount" />
+  </joint>
+  <joint name="front_mount_joint" type="fixed">
+    <origin xyz="0.080 0 0" rpy="0 0 0" />
+    <parent link="front_b_mount"/>
+    <child link="front_mount" />
+  </joint>
+  <joint name="rear_c_mount_joint" type="fixed">
+    <origin xyz="-0.040 0 0.064263" rpy="0 0 0" />
+    <parent link="chassis_link"/>
+    <child link="rear_c_mount" />
+  </joint>
+  <joint name="rear_b_mount_joint" type="fixed">
+    <origin xyz="-0.080 0 0" rpy="0 0 0" />
+    <parent link="rear_c_mount"/>
+    <child link="rear_b_mount" />
+  </joint>
+  <joint name="rear_moint_joint" type="fixed">
+    <origin xyz="-0.080 0 0" rpy="0 0 0" />
+    <parent link="rear_b_mount"/>
+    <child link="rear_mount" />
+  </joint>
   <!--
     Mounting point for accessories on the front bumper.

File: dingo_description/urdf/dingo-o.urdf.xacro (robot description, xacro)
@@ -121,48 +121,46 @@
       - rear
   -->
-  <xacro:unless value="${pacs_enabled}">
-    <link name="front_mount"/>
-    <link name="front_b_mount"/>
-    <link name="front_c_mount"/>
-    <link name="rear_mount"/>
-    <link name="rear_b_mount"/>
-    <link name="rear_c_mount"/>
-    <link name="mid_mount"/>
-    <joint name="mid_mount_joint" type="fixed">
-      <origin xyz="0 0 0.069023" rpy="0 0 0" />
-      <parent link="chassis_link"/>
-      <child link="mid_mount" />
-    </joint>
-    <joint name="front_c_mount_joint" type="fixed">
-      <origin xyz="0.080 0 0" rpy="0 0 0" />
-      <parent link="mid_mount"/>
-      <child link="front_c_mount" />
-    </joint>
-    <joint name="front_b_mount_joint" type="fixed">
-      <origin xyz="0.080 0 0" rpy="0 0 0" />
-      <parent link="front_c_mount"/>
-      <child link="front_b_mount" />
-    </joint>
-    <joint name="front_mount_joint" type="fixed">
-      <origin xyz="0.080 0 0" rpy="0 0 0" />
-      <parent link="front_b_mount"/>
-      <child link="front_mount" />
-    </joint>
-    <joint name="rear_c_mount_joint" type="fixed">
-      <origin xyz="-0.080 0 0" rpy="0 0 0" />
-      <parent link="mid_mount"/>
-      <child link="rear_c_mount" />
-    </joint>
-    <joint name="rear_b_mount_joint" type="fixed">
-      <origin xyz="-0.080 0 0" rpy="0 0 0" />
-      <parent link="rear_c_mount"/>
-      <child link="rear_b_mount" />
-    </joint>
-    <joint name="rear_moint_joint" type="fixed">
-      <origin xyz="-0.080 0 0" rpy="0 0 0" />
-      <parent link="rear_b_mount"/>
-      <child link="rear_mount" />
-    </joint>
-  </xacro:unless>
+  <link name="front_mount"/>
+  <link name="front_b_mount"/>
+  <link name="front_c_mount"/>
+  <link name="rear_mount"/>
+  <link name="rear_b_mount"/>
+  <link name="rear_c_mount"/>
+  <link name="mid_mount"/>
+  <joint name="mid_mount_joint" type="fixed">
+    <origin xyz="0 0 0.069023" rpy="0 0 0" />
+    <parent link="chassis_link"/>
+    <child link="mid_mount" />
+  </joint>
+  <joint name="front_c_mount_joint" type="fixed">
+    <origin xyz="0.080 0 0" rpy="0 0 0" />
+    <parent link="mid_mount"/>
+    <child link="front_c_mount" />
+  </joint>
+  <joint name="front_b_mount_joint" type="fixed">
+    <origin xyz="0.080 0 0" rpy="0 0 0" />
+    <parent link="front_c_mount"/>
+    <child link="front_b_mount" />
+  </joint>
+  <joint name="front_mount_joint" type="fixed">
+    <origin xyz="0.080 0 0" rpy="0 0 0" />
+    <parent link="front_b_mount"/>
+    <child link="front_mount" />
+  </joint>
+  <joint name="rear_c_mount_joint" type="fixed">
+    <origin xyz="-0.080 0 0" rpy="0 0 0" />
+    <parent link="mid_mount"/>
+    <child link="rear_c_mount" />
+  </joint>
+  <joint name="rear_b_mount_joint" type="fixed">
+    <origin xyz="-0.080 0 0" rpy="0 0 0" />
+    <parent link="rear_c_mount"/>
+    <child link="rear_b_mount" />
+  </joint>
+  <joint name="rear_moint_joint" type="fixed">
+    <origin xyz="-0.080 0 0" rpy="0 0 0" />
+    <parent link="rear_b_mount"/>
+    <child link="rear_mount" />
+  </joint>
   <!--
     Mounting point for accessories on the front bumper.

File: dingo_description/urdf/pacs.urdf.xacro (robot description, xacro)
@@ -280,5 +280,5 @@
     <xacro:property name="omni" value="$(optenv DINGO_OMNI 0)"/>
     <xacro:property name="riser" value="$(optenv DINGO_PACS_RISER 0)"/>
-    <xacro:property name="pacs_enabled" value="$(optenv DINGO_PACS_ENABLED 1)" />
+    <xacro:property name="pacs_enabled" value="$(optenv DINGO_PACS_ENABLED 0)" />
     <xacro:if value="${pacs_enabled}">
       <xacro:property name="riser_x" value="0.0"/>
@@ -291,6 +291,6 @@
         </xacro:riser>
       </xacro:if>
+      <xacro:base_mounts parent="chassis_link" omni="${omni}"/>
     </xacro:if>
-    <xacro:base_mounts parent="chassis_link" omni="${omni}"/>
   </xacro:macro>
 </robot>
